Commit message: Updated the DensoVS060 model to fix it. Updated the swift plotting support keboard control function to make it cleaner. Updated the version number in the toml file in preparation for the next release.

File: ir_support/robots/DensoVS060/DensoVS060.urdf (robot description, URDF)
Before this commit: robot DensoVS060v3, 7 links, 6 joints
Links:
- added link link1b
Joints:
- added joint link1_to_link1b: type fixed, parent link1, child link1b, origin xyz=0 0 0 rpy=-1.5708 0 0
- joint joint2: origin xyz=0 0 0 rpy=1.5708 0 0 -> xyz=0 0 0 rpy=0 0 -3.1416; parent link1 -> link1b
